File: elec/layout/default/sgp40-d-r4.kicad_pcb (KiCad board)
At the start: 2 copper layers, 225.7 x 100.8 mm, 0 parts

Commit message: layout
Parts:
- added C1: Multilayer Ceramic Capacitors MLCC - SMD/SMT 1uF 6.3V 0402 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, lib:C0402, F.Cu at (161.6, 101.0)
- added C2: Multilayer Ceramic Capacitors MLCC - SMD/SMT 1uF 6.3V 0402 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, lib:C0402, F.Cu at (157.2, 100.0)
- added U1: , lib:DFN-6_L2.4-W2.4-P0.80-TL-EP, F.Cu at (159.4, 100.5)
Routing:
- net gnd: track 0.00 -> 4.89 mm
- net vcc: track 0.00 -> 2.30 mm
Changed lines of the file:
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@@
   )
   (net 0 "")
+  (net 1 "vcc")
+  (net 2 "gnd")
+  (net 3 "sda")
+  (net 4 "scl")
+  (footprint "lib:DFN-6_L2.4-W2.4-P0.80-TL-EP" (layer "F.Cu")
+    (at 159.395 100.55)
+    (attr smd)
+    (fp_text reference "U1" (at 0 -4.8) (layer "F.SilkS")
+        (effects (font (size 1 1) (thickness 0.15)))
+    )
+    (fp_text value "" (at 0 4.8) (layer "F.Fab")
+        (effects (font (size 1 1) (thickness 0.15)))
+    )
+    (fp_text user "${REFERENCE}" (at 0 0) (layer "F.Fab")
+        (effects (font (size 1 1) (thickness 0.15)))
+    )
+    (fp_line (start -1.3 -1.3) (end 1.3 -1.3)
+      (stroke (width 0.15) (type solid)) (layer "F.SilkS"))
+    (fp_line (start -1.3 1.3) (end 1.3 1.3)
+      (stroke (width 0.15) (type solid)) (layer "F.SilkS"))
+    (fp_circle (center -1.7 -0.7) (end -1.6 -0.7)
+      (stroke (width 0.1) (type solid)) (fill none) (layer "F.SilkS"))
+    (fp_circle (center -1.4 -1) (end -1.3 -1)
+      (stroke (width 0.2) (type solid)) (fill none) (layer "Cmts.User"))
+    (fp_circle (center -1.22 -1.22) (end -1.19 -1.22)
+      (stroke (width 0.06) (type solid)) (fill none) (layer "F.Fab"))
+    (pad "1" smd rect (at -1.14 -0.8) (size 0.58 0.45) (layers "F.Cu" "F.Paste" "F.Mask")
+      (net 1 "vcc") (pintype "stereo"))
+    (pad "2" smd rect (at -1.14 0) (size 0.58 0.45) (layers "F.Cu" "F.Paste" "F.Mask")
+      (net 2 "gnd") (pintype "stereo"))
+    (pad "3" smd rect (at -1.14 0.8) (size 0.58 0.45) (layers "F.Cu" "F.Paste" "F.Mask")
+      (net 3 "sda") (pintype "stereo"))
+    (pad "4" smd rect (at 1.14 0.8) (size 0.58 0.45) (layers "F.Cu" "F.Paste" "F.Mask")
+      (net 2 "gnd") (pintype "stereo"))
+    (pad "5" smd rect (at 1.14 0) (size 0.58 0.45) (layers "F.Cu" "F.Paste" "F.Mask")
+      (net 1 "vcc") (pintype "stereo"))
+    (pad "6" smd rect (at 1.14 -0.8) (size 0.58 0.45) (layers "F.Cu" "F.Paste" "F.Mask")
+      (net 4 "scl") (pintype "stereo"))
+    (pad "7" smd rect (at 0 0) (size 1.25 1.65) (layers "F.Cu" "F.Paste" "F.Mask")
+      (net 2 "gnd") (pintype "stereo"))
+    (model "/Users/narayanpowderly/Documents/atopile-workspace/the-everything-sensor/.ato/modules/sgp40-d-r4/elec/footprints/footprints.3dshapes/DFN-6_L2.4-W2.4-P0.80-TL-EP.wrl"
+      (offset (xyz 0 -0 -0))
+      (scale (xyz 1 1 1))
+      (rotate (xyz 0 0 0))
+    )
+  )
+  (footprint "lib:C0402" (layer "F.Cu")
+    (at 157.151861 100.00701 -90)
+    (descr "Capacitor SMD 0402 (1005 Metric), square (rectangular) end terminal, IPC_7351 nominal, (Body size source: IPC-SM-782 page 76, https://www.pcb-3d.com/wordpress/wp-content/uploads/ipc-sm-782a_amendment_1_and_2.pdf), generated with kicad-footprint-generator")
+    (tags "capacitor")
+    (attr smd)
+    (fp_text reference "C2" (at 0 -1.16 90) (layer "F.SilkS")
+        (effects (font (size 1 1) (thickness 0.15)))
+    )
+    (fp_text value "Multilayer Ceramic Capacitors MLCC - SMD/SMT 1uF 6.3V 0402 RoHS" (at 0 1.16 90) (layer "F.Fab")
+        (effects (font (size 1 1) (thickness 0.15)))
+    )
+    (fp_text user "${REFERENCE}" (at 0 0 90) (layer "F.Fab")
+        (effects (font (size 0.25 0.25) (thickness 0.04)))
+    )
+    (fp_line (start -0.107836 -0.36) (end 0.107836 -0.36)
+      (stroke (width 0.12) (type solid)) (layer "F.SilkS"))
+    (fp_line (start -0.107836 0.36) (end 0.107836 0.36)
+      (stroke (width 0.12) (type solid)) (layer "F.SilkS"))
+    (fp_line (start -0.91 -0.46) (end 0.91 -0.46)
+      (stroke (width 0.05) (type solid)) (layer "F.CrtYd"))
+    (fp_line (start -0.91 0.46) (end -0.91 -0.46)
+      (stroke (width 0.05) (type solid)) (layer "F.CrtYd"))
+    (fp_line (start 0.91 -0.46) (end 0.91 0.46)
+      (stroke (width 0.05) (type solid)) (layer "F.CrtYd"))
+    (fp_line (start 0.91 0.46) (end -0.91 0.46)
+      (stroke (width 0.05) (type solid)) (layer "F.CrtYd"))
+    (fp_line (start -0.5 -0.25) (end 0.5 -0.25)
+      (stroke (width 0.1) (type solid)) (layer "F.Fab"))
+    (fp_line (start -0.5 0.25) (end -0.5 -0.25)
+      (stroke (width 0.1) (type solid)) (layer "F.Fab"))
+    (fp_line (start 0.5 -0.25) (end 0.5 0.25)
+      (stroke (width 0.1) (type solid)) (layer "F.Fab"))
+    (fp_line (start 0.5 0.25) (end -0.5 0.25)
+      (stroke (width 0.1) (type solid)) (layer "F.Fab"))
+    (pad "1" smd roundrect (at -0.48 0 270) (size 0.56 0.62) (layers "F.Cu" "F.Paste" "F.Mask") (roundrect_rratio 0.25)
+      (net 1 "vcc") (pintype "stereo"))
+    (pad "2" smd roundrect (at 0.48 0 270) (size 0.56 0.62) (layers "F.Cu" "F.Paste" "F.Mask") (roundrect_rratio 0.25)
+      (net 2 "gnd") (pintype "stereo"))
+    (model "${KICAD6_3DMODEL_DIR}/Capacitor_SMD.3dshapes/C_0402_1005Metric.wrl"
+      (offset (xyz 0 0 0))
+      (scale (xyz 1 1 1))
+      (rotate (xyz 0 0 0))
+    )
+  )
+  (footprint "lib:C0402" (layer "F.Cu")
+    (at 161.628696 101.013782 -90)
+    (descr "Capacitor SMD 0402 (1005 Metric), square (rectangular) end terminal, IPC_7351 nominal, (Body size source: IPC-SM-782 page 76, https://www.pcb-3d.com/wordpress/wp-content/uploads/ipc-sm-782a_amendment_1_and_2.pdf), generated with kicad-footprint-generator")
+    (tags "capacitor")
+    (attr smd)
+    (fp_text reference "C1" (at 0 -1.16 90) (layer "F.SilkS")
+        (effects (font (size 1 1) (thickness 0.15)))
+    )
+    (fp_text value "Multilayer Ceramic Capacitors MLCC - SMD/SMT 1uF 6.3V 0402 RoHS" (at 0 1.16 90) (layer "F.Fab")
+        (effects (font (size 1 1) (thickness 0.15)))
+    )
+    (fp_text user "${REFERENCE}" (at 0 0 90) (layer "F.Fab")
+        (effects (font (size 0.25 0.25) (thickness 0.04)))
+    )
+    (fp_line (start -0.107836 -0.36) (end 0.107836 -0.36)
+      (stroke (width 0.12) (type solid)) (layer "F.SilkS"))
+    (fp_line (start -0.107836 0.36) (end 0.107836 0.36)
+      (stroke (width 0.12) (type solid)) (layer "F.SilkS"))
+    (fp_line (start -0.91 -0.46) (end 0.91 -0.46)
+      (stroke (width 0.05) (type solid)) (layer "F.CrtYd"))
+    (fp_line (start -0.91 0.46) (end -0.91 -0.46)
+      (stroke (width 0.05) (type solid)) (layer "F.CrtYd"))
+    (fp_line (start 0.91 -0.46) (end 0.91 0.46)
+      (stroke (width 0.05) (type solid)) (layer "F.CrtYd"))
+    (fp_line (start 0.91 0.46) (end -0.91 0.46)
+      (stroke (width 0.05) (type solid)) (layer "F.CrtYd"))
+    (fp_line (start -0.5 -0.25) (end 0.5 -0.25)
+      (stroke (width 0.1) (type solid)) (layer "F.Fab"))
+    (fp_line (start -0.5 0.25) (end -0.5 -0.25)
+      (stroke (width 0.1) (type solid)) (layer "F.Fab"))
+    (fp_line (start 0.5 -0.25) (end 0.5 0.25)
+      (stroke (width 0.1) (type solid)) (layer "F.Fab"))
+    (fp_line (start 0.5 0.25) (end -0.5 0.25)
+      (stroke (width 0.1) (type solid)) (layer "F.Fab"))
+    (pad "1" smd roundrect (at -0.48 0 270) (size 0.56 0.62) (layers "F.Cu" "F.Paste" "F.Mask") (roundrect_rratio 0.25)
+      (net 1 "vcc") (pintype "stereo"))
+    (pad "2" smd roundrect (at 0.48 0 270) (size 0.56 0.62) (layers "F.Cu" "F.Paste" "F.Mask") (roundrect_rratio 0.25)
+      (net 2 "gnd") (pintype "stereo"))
+    (model "${KICAD6_3DMODEL_DIR}/Capacitor_SMD.3dshapes/C_0402_1005Metric.wrl"
+      (offset (xyz 0 0 0))
+      (scale (xyz 1 1 1))
+      (rotate (xyz 0 0 0))
+    )
+  )
   (gr_circle (center 225.62 81.79) (end 227.32 81.79)
     (stroke (width 0.1) (type solid)) (fill none) (layer "Edge.Cuts"))
@@
       (xy 69.100734 49.778315)
     )
-    (stroke (width 0) (type solid)) (fill none) (layer "Edge.Cuts"))
+    (stroke (width 0.1) (type solid)) (fill none) (layer "Edge.Cuts"))
   (gr_arc (start 261.62 113.79) (mid 260.448427 116.618427) (end 257.62 117.79)
     (stroke (width 0.1) (type solid)) (layer "Edge.Cuts"))
@@
     (effects (font (size 2 2) (thickness 0.1)) (justify left bottom))
   )
+  (segment (start 160.551218 100.533782) (end 160.535 100.55) (width 0.25) (layer "F.Cu") (net 1))
+  (segment (start 157.151861 99.52701) (end 158.03201 99.52701) (width 0.25) (layer "F.Cu") (net 1))
+  (segment (start 158.03201 99.52701) (end 158.255 99.75) (width 0.25) (layer "F.Cu") (net 1))
+  (segment (start 161.628696 100.533782) (end 160.551218 100.533782) (width 0.25) (layer "F.Cu") (net 1))
+  (segment (start 160.535 101.35) (end 160.195 101.35) (width 0.25) (layer "F.Cu") (net 2))
+  (segment (start 161.628696 101.493782) (end 160.678782 101.493782) (width 0.25) (layer "F.Cu") (net 2))
+  (segment (start 159.395 100.55) (end 158.255 100.55) (width 0.25) (layer "F.Cu") (net 2))
+  (segment (start 157.151861 100.48701) (end 158.19201 100.48701) (width 0.25) (layer "F.Cu") (net 2))
+  (segment (start 160.195 101.35) (end 159.395 100.55) (width 0.25) (layer "F.Cu") (net 2))
+  (segment (start 158.19201 100.48701) (end 158.255 100.55) (width 0.25) (layer "F.Cu") (net 2))
+  (segment (start 160.678782 101.493782) (end 160.535 101.35) (width 0.25) (layer "F.Cu") (net 2))
   (group "" (id 6c1ef9f7-0f34-47bb-ac1a-76df23fb396e)
     (members
